File: Schematics/upper_lc_board/modules/ESP_breakout_module/ESP_breakout_module.kicad_sch (KiCad schematic)
At the start: 24 parts, among them J8 USB_C_Female_USB2_Small, SW1 SW_ESP_BOOT_MODE, SW2 SW_ESP_RESET, U1 ESP32-S3-WROOM-1-N16, U2 ISO1044BDR

Commit message: add relative datasheets to symbol fields
Parts:
- D4: now left out of the parts list
Changed lines of the file:
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@@
 			)
 		)
-		(property "Datasheet" "https://www.usb.org/sites/default/files/documents/usb_type-c.zip"
+		(property "Datasheet" "${KIPRJMOD}/../../Datasheets/USBSC-conn.pdf"
 			(at 154.94 113.03 0)
 			(effects
@@
 			)
 		)
-		(property "Datasheet" "https://www.espressif.com/sites/default/files/documentation/esp32-s3-wroom-1_wroom-1u_datasheet_en.pdf"
+		(property "Datasheet" "${KIPRJMOD}/../../Datasheets/MCU-esp32-s3-wroom-1_wroom-1u_datasheet_en.pdf"
 			(at 92.71 88.9 0)
 			(effects
@@
 		(unit 1)
 		(exclude_from_sim no)
-		(in_bom yes)
+		(in_bom no)
 		(on_board yes)
 		(dnp no)
@@
 			)
 		)
-		(property "Datasheet" "https://cdn-shop.adafruit.com/datasheets/WS2812B.pdf"
+		(property "Datasheet" "${KIPRJMOD}/../../Datasheets/LED-WS2812B.pdf"
 			(at 119.38 169.545 0)
 			(effects
@@
 			)
 		)
-		(property "Datasheet" "https://datasheet.lcsc.com/lcsc/2304140030_XKB-Connection-TS-1187A-B-A-B_C318884.pdf"
+		(property "Datasheet" "${KIPRJMOD}/../../Datasheets/buttons-modeselec.pdf"
 			(at 156.21 39.37 0)
 			(effects
@@
 			)
 		)
-		(property "Datasheet" "https://www.ti.com/lit/ds/symlink/iso1044.pdf"
+		(property "Datasheet" "${KIPRJMOD}/../../Datasheets/CAN-T_ISO1044.pdf"
 			(at 215.9 67.31 0)
 			(effects
@@
 			)
 		)
-		(property "Datasheet" "https://datasheet.lcsc.com/lcsc/2304140030_XKB-Connection-TS-1187A-B-A-B_C318884.pdf"
+		(property "Datasheet" "${KIPRJMOD}/../../Datasheets/buttons-modeselec.pdf"
 			(at 156.21 57.15 0)
 			(effects
